Commit message: 四轮模型

File: robot_description_py/install/robot_description_py/share/robot_description_py/urdf/robot_base.urdf (robot description, URDF)
Before this commit: robot shakimabot, 2 links, 1 joints
Links:
- added link imu_link; visual box size=0.02 0.02 0.02
- added link left_wheel_1_link; visual cylinder length=0.04 radius=0.032
- added link left_wheel_2_link; visual cylinder length=0.04 radius=0.032
- added link odom
- added link right_wheel_1_link; visual cylinder length=0.04 radius=0.032
- added link right_wheel_2_link; visual cylinder length=0.04 radius=0.032
- link laser_link: geometry visual cylinder length=0.04 radius=0.03
Joints:
- added joint base_joint: type fixed, parent odom, child base_link, origin xyz=0.0 0.0 0.075 rpy=0 0 0
- added joint imu_joint: type fixed, parent base_link, child imu_link, origin xyz=0 0 0.02
- added joint left_wheel_1_joint: type continuous, parent base_link, child left_wheel_1_link, origin xyz=-0.14 0.14 -0.06, axis 0 1 0
- added joint left_wheel_2_joint: type continuous, parent base_link, child left_wheel_2_link, origin xyz=0.14 0.14 -0.06, axis 0 1 0
- added joint right_wheel_1_joint: type continuous, parent base_link, child right_wheel_1_link, origin xyz=-0.14 -0.14 -0.06, axis 0 1 0
- added joint right_wheel_2_joint: type continuous, parent base_link, child right_wheel_2_link, origin xyz=0.14 -0.14 -0.06, axis 0 1 0
- joint laser_joint: origin xyz=0 0 0.075 -> xyz=0 0 0.08
