Commit message: 完成建模和调参控制

File: robot_description_py/urdf/robot_base.urdf (robot description, URDF)
Before this commit: robot shakimabot, 8 links, 7 joints
Links:
- removed link left_wheel_1_link
- removed link left_wheel_2_link
- removed link right_wheel_1_link
- removed link right_wheel_2_link
- added link left_back_wheel_link; visual cylinder length=0.04 radius=0.032
- added link left_front_wheel_link; visual cylinder length=0.04 radius=0.032
- added link right_back_wheel_link; visual cylinder length=0.04 radius=0.032
- added link right_front_wheel_link; visual cylinder length=0.04 radius=0.032
Joints:
- removed joint left_wheel_1_joint
- removed joint left_wheel_2_joint
- removed joint right_wheel_1_joint
- removed joint right_wheel_2_joint
- added joint left_back_wheel_joint: type continuous, parent base_link, child left_back_wheel_link, origin xyz=-0.14 0.14 -0.06, axis 0 1 0
- added joint left_front_wheel_joint: type continuous, parent base_link, child left_front_wheel_link, origin xyz=0.14 0.14 -0.06, axis 0 1 0
- added joint right_back_wheel_joint: type continuous, parent base_link, child right_back_wheel_link, origin xyz=-0.14 -0.14 -0.06, axis 0 1 0
- added joint right_front_wheel_joint: type continuous, parent base_link, child right_front_wheel_link, origin xyz=0.14 -0.14 -0.06, axis 0 1 0

Commit message: 舵轮模型完成

File: robot_description_py/urdf/robot_base.urdf (robot description, URDF)
Before this commit: robot shakimabot, 8 links, 7 joints
Links:
- added link left_back_wheel_mount_link; visual box size=0.02 0.02 0.04
- added link left_front_wheel_mount_link; visual box size=0.02 0.02 0.04
- added link right_back_wheel_mount_link; visual box size=0.02 0.02 0.04
- added link right_front_wheel_mount_link; visual box size=0.02 0.02 0.04
Joints:
- added joint left_back_wheel_mount_joint: type continuous, parent base_link, child left_back_wheel_mount_link, origin xyz=-0.14 0.12 -0.08, axis 0 0 1
- added joint left_front_wheel_mount_joint: type continuous, parent base_link, child left_front_wheel_mount_link, origin xyz=0.14 0.12 -0.08, axis 0 0 1
- added joint right_back_wheel_mount_joint: type continuous, parent base_link, child right_back_wheel_mount_link, origin xyz=-0.14 -0.12 -0.08, axis 0 0 1
- added joint right_front_wheel_mount_joint: type continuous, parent base_link, child right_front_wheel_mount_link, origin xyz=0.14 -0.12 -0.08, axis 0 0 1
- joint base_joint: origin xyz=0.0 0.0 0.075 rpy=0 0 0 -> xyz=0.0 0.0 0.13 rpy=0 0 0
- joint left_back_wheel_joint: origin xyz=-0.14 0.14 -0.06 -> xyz=0 0 -0.03; parent base_link -> left_back_wheel_mount_link
- joint left_front_wheel_joint: origin xyz=0.14 0.14 -0.06 -> xyz=0 0 -0.03; parent base_link -> left_front_wheel_mount_link
- joint right_back_wheel_joint: origin xyz=-0.14 -0.14 -0.06 -> xyz=0 0 -0.03; parent base_link -> right_back_wheel_mount_link
- joint right_front_wheel_joint: origin xyz=0.14 -0.14 -0.06 -> xyz=0 0 -0.03; parent base_link -> right_front_wheel_mount_link

Commit message: 添加了gazebo的描述xml

File: robot_description_py/urdf/robot_base.urdf (robot description, URDF)
Before this commit: robot shakimabot, 12 links, 11 joints
Links:
- removed link odom
- added link odom_
- link base_link: mass None -> 1; geometry collision box size=0.36 0.24 0.12; visual box size=0.36 0.24 0.12
- link imu_link: mass None -> 0.1; geometry collision box size=0.02 0.02 0.02; visual box size=0.02 0.02 0.02
- link laser_link: mass None -> 0.1; geometry collision cylinder length=0.04 radius=0.03; visual cylinder length=0.04 radius=0.03
- link left_back_wheel_link: mass None -> 0.2; geometry collision cylinder length=0.04 radius=0.032; visual cylinder length=0.04 radius=0.032
- link left_back_wheel_mount_link: mass None -> 0.1; geometry collision box size=0.02 0.02 0.04; visual box size=0.02 0.02 0.04
- link left_front_wheel_link: mass None -> 0.2; geometry collision cylinder length=0.04 radius=0.032; visual cylinder length=0.04 radius=0.032
- link left_front_wheel_mount_link: mass None -> 0.1; geometry collision box size=0.02 0.02 0.04; visual box size=0.02 0.02 0.04
- link right_back_wheel_link: mass None -> 0.2; geometry collision cylinder length=0.04 radius=0.032; visual cylinder length=0.04 radius=0.032
- link right_back_wheel_mount_link: mass None -> 0.1; geometry collision box size=0.02 0.02 0.04; visual box size=0.02 0.02 0.04
- link right_front_wheel_link: mass None -> 0.2; geometry collision cylinder length=0.04 radius=0.032; visual cylinder length=0.04 radius=0.032
- link right_front_wheel_mount_link: mass None -> 0.1; geometry collision box size=0.02 0.02 0.04; visual box size=0.02 0.02 0.04
Joints:
- joint base_joint: parent odom -> odom_
